File: schematics/fc-ee/fc-ee.kicad_sch (KiCad schematic)
At the start: 17 parts, among them J1 USB_B_Micro, SW1 SW_SPDT, U1 STM32F407VETx, X1 8MHz

Commit message: update 2/25/26
Parts:
- added C10: 10n, symbol Device:C
- added C11, C12, C14: 0.1u, symbol Device:C
- added C13: 1u, symbol Device:C
- added D1, D3: LED, symbol Device:LED
- added R4, R5, R6, R7: 10k, symbol Device:R_Small
- added R8, R9: 1k, symbol Device:R_Small
- added U2: MPU-9250, Sensor_Motion:InvenSense_QFN-24_3x3mm_P0.4mm, symbol Sensor_Motion:MPU-9250
Connections:
- net GYRO_SDA is gone; now on an unnamed net: U1.32 (PA7)
- net +3.3V: now also C10.2, C12.1, U2.13 (VDD), U2.8 (VDDIO)
- net GND: now also C11.1, C13.2, C14.2, D1.1 (K), D3.1 (K), R5.1, U2.11 (FSYNC), U2.18 (GND), U2.20 (RESV_GND)
- net GYRO_INT: now also U2.12 (INT)
- net GYRO_SCL: now also U2.23 (SCL/SCLK)
- net GYRO_SDO: now also U2.9 (AD0/MISO)
- net LED1: now also R8.1
- net LED2: now also R9.1
- net SCL_PAD: now also R6.2; no longer U1.92 (PB6)
- net SDA_PAD: now also R7.2; no longer U1.93 (PB7)
- net USB_5V: now also R4.2, R5.2; no longer J1.1 (VBUS)
- net at U1.29 (PA4), U1.47 (PB10): now also U2.22 (~{CS}), U2.24 (SDA/MOSI)
- new net: C10.1, C11.2
- new net: C12.2, C13.1
- new net: C14.1, U2.10 (REGOUT)
- new net: R6.1, U1.92 (PB6)
- new net: R7.1, U1.93 (PB7)
- new net: J1.1 (VBUS), R4.1
- new net: D1.2 (A), R8.2
- new net: D3.2 (A), R9.2
- no-connect marks 2 -> 4

Commit message: update 2/26/26
Parts:
- added C15, C16: 22u, symbol Device:C
- added C17, C18: 100n, symbol Device:C
- added D2: LED, symbol Device:LED
- added J2, J3, J4: Conn_01x04_Pin, symbol Connector:Conn_01x04_Pin
- added R10: 1k, symbol Device:R_Small
- added U3: AMS1117-3.3, Package_TO_SOT_SMD:SOT-223-3_TabPin2, symbol Regulator_Linear:AMS1117-3.3
Connections:
- net USART5_TX is gone; now on net USART6_RX: U1.64 (PC7)
- net +3.3V: now also J2.4 (Pin_4), J3.4 (Pin_4), J4.4 (Pin_4)
- net +3.3VA: now also U1.21 (VREF+)
- net GND: now also C15.2, C16.2, C17.1, C18.1, J2.1 (Pin_1), J3.1 (Pin_1), J4.1 (Pin_1), R10.1, U3.1 (GND)
- net USART1_RX: now also J4.2 (Pin_2)
- net USART1_TX: now also J4.3 (Pin_3)
- net USART3_RX: now also J3.2 (Pin_2)
- net USART6_RX: now also J2.2 (Pin_2); no longer U1.63 (PC6)
- net USB_5V: now also J1.1 (VBUS), R4.1, C15.1, U3.3 (VI); no longer R4.2, U1.34 (PC5)
- net at U1.29 (PA4), U1.32 (PA7), U1.47 (PB10)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: now also J3.3 (Pin_3)
- net at U1.49 (VCAP_1): now also C17.2
- net at U1.73 (VCAP_2): now also C18.2
- new net: R4.2, U1.34 (PC5)
- new net +3.3v: C16.1, D2.2 (A), U3.2 (VO)
- new net PWR_LED_K: D2.1 (K), R10.2
- new net USART6_TX: J2.3 (Pin_3), U1.63 (PC6)
- no-connect marks 4 -> 60
Other:
- note added: "CoreSen Flight Computer v1"
- note added: "IMU (MPU9250)"
- note added: "LED (from STM line)"
- note added: "Linear Regulator (ASM1117-3.3v)"
- note added: "MICROCONTROLLER(& USB)"
- note added: "The higher voltage comes from the USB and outputs as +3.3v which is supplied to the rest of the components"
- note added: "We can use serial-wire debug on PA13&14"
- title: (none) -> CoreSen-FC1
- moved on the sheet: C1, C10, C11, C12, C13, C14, C2, C3, C4, C5, C6, C7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

Commit message: 3/1/26
Parts:
- removed X1: 8MHz, symbol Device:Crystal_GND2_Small
- added C19, C20: 22u, Capacitor_SMD:C_0805_2012Metric, symbol Device:C
- added C21, C22: 10p, Capacitor_SMD:C_0603_1608Metric, symbol Device:C
- added D5: BAT54C, Package_TO_SOT_SMD:SOT-23, symbol Diode:BAT54C
- added J5: Conn_01x03_Pin, Connector_JST:JST_NV_B03P-NV_1x03_P5.00mm_Vertical, symbol Connector:Conn_01x03_Pin
- added TP1, TP2, TP3, TP4, TP5, TP6: TestPoint, TestPoint:TestPoint_Pad_D4.0mm, symbol Connector:TestPoint
- added U4: AMS1117-5.0, Package_TO_SOT_SMD:SOT-223-3_TabPin2, symbol Regulator_Linear:AMS1117-5.0
- added Y1: 8MHz, Crystal:Crystal_SMD_3225-4Pin_3.2x2.5mm_HandSoldering, symbol Device:Crystal_GND24_Small
- C1, C13, C17, C18, C2, C3, C4, C7, C8, C9: footprint (none) -> Capacitor_SMD:C_0402_1005Metric
- C10, C5, C6: footprint (none) -> Capacitor_SMD:C_0603_1608Metric
- C11, C12, C14: value 0.1u -> 100n; footprint (none) -> Capacitor_SMD:C_0402_1005Metric
- C15, C16: footprint (none) -> Capacitor_SMD:C_0805_2012Metric
- D1, D2, D3: footprint (none) -> LED_SMD:LED_0201_0603Metric
- FB1: footprint (none) -> Inductor_SMD:L_0603_1608Metric
- J1: footprint (none) -> Connector_USB:USB_Micro-B_Molex_47346-0001
- J2, J3, J4: footprint (none) -> Connector_PinHeader_2.00mm:PinHeader_1x04_P2.00mm_Vertical
- R1, R10, R2, R3, R4, R5, R6, R7, R8, R9: footprint (none) -> Resistor_SMD:R_0402_1005Metric
- SW1: footprint (none) -> Button_Switch_THT:SW_E-Switch_EG1224_SPDT_Angled
Connections:
- net +3.3v is gone; now on net +3.3V: C16.1, D2.2 (A), U3.2 (VO)
- net +3.3V: now also U2.1 (RESV_VDDIO), J5.3 (Pin_3)
- net BUZZER: now also TP1.1
- net CURRENT_PAD: now also TP6.1
- net GND: now also C19.2, C20.2, C21.2, C22.2, J5.1 (Pin_1), U4.1 (GND), Y1.2, Y1.4
- net PPM_IN: now also J5.2 (Pin_2)
- net RCC_OSC_IN: now also C21.1, Y1.1
- net RCC_OSC_OUT: now also C22.1, Y1.3
- net RSSI_PAD: now also TP5.1
- net SCL_PAD: now also TP2.1
- net SDA_PAD: now also TP3.1
- net USB_5V: now also D5.2; no longer C15.1, U3.3 (VI)
- net VBAT_PAD: now also TP4.1
- new net: C15.1, D5.3, U3.3 (VI)
- new net +5V: C20.1, D5.1, U4.2 (VO)
- new net GYRO_CS: U1.29 (PA4), U2.22 (~{CS})
- new net GYRO_SDA: U1.32 (PA7), U2.24 (SDA/MOSI)
- new net USART3_TX: J3.3 (Pin_3), U1.47 (PB10)
- new net VDC: C19.1, U4.3 (VI)
- no-connect marks 60 -> 61
Other:
- note added: "5V regulator that steps down the higher voltage from the battery to 5v for 3.3v conversion and other components"
- note added: "Linear Regulator (ASM1117-5v)"
- note added: "Linear Regulators(5V & 3V)"
- note added: "The higher voltage comes from the USB/BAT->5V converter above and outputs as +3.3v which is supplied to the rest of the components"
- note removed: "The higher voltage comes from the USB and outputs as +3.3v which is supplied to the rest of the components"
- moved on the sheet: C15, C16, D1, D2, D3, R10, R8, R9, U3
